Commit message: Pushing all novelties, as urdf files and minor changes

File: robots/z1_description/urdf/z1.urdf (robot description, URDF)
Before this commit: robot z1_description, 10 links, 9 joints
Links:
- link gripperMover: geometry collision mesh filename=package://robots/z1_description/meshes/collision/z1_Gripper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 scale=1 1 1; visual mesh filename=package://robots/z1_description/meshes/visual/z1_GripperMov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 scale=1 1 1
- link gripperStator: geometry collision mesh filename=package://robots/z1_description/meshes/collision/z1_Gripper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 scale=1 1 1; visual mesh filename=package://robots/z1_description/meshes/visual/z1_GripperSta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 scale=1 1 1
- link link00: geometry collision cylinder length=0.051 radius=0.0325; visual mesh filename=package://robots/z1_description/meshes/visual/z1_Link00.dae scale=1 1 1
- link link01: geometry visual mesh filename=package://robots/z1_description/meshes/visual/z1_Link01.dae scale=1 1 1
- link link02: geometry collision cylinder length=0.051 radius=0.0325; collision cylinder length=0.102 radius=0.0325
- link link03: geometry collision cylinder length=0.059 radius=0.0325; collision cylinder length=0.116 radius=0.02
- link link04: geometry collision cylinder length=0.067 radius=0.0325; visual mesh filename=package://robots/z1_description/meshes/visual/z1_Link04.dae scale=1 1 1
- link link05: geometry visual mesh filename=package://robots/z1_description/meshes/visual/z1_Link05.dae scale=1 1 1
- link link06: geometry collision cylinder length=0.051 radius=0.0325; visual mesh filename=package://robots/z1_description/meshes/visual/z1_Link06.dae scale=1 1 1
Joints:
- joint joint1: limit lower=-2.6179938779914944 upper=2.6179938779914944 effort=30.0 velocity=3.1415 -> lower=-2.6179938779914944 upper=2.6179938779914944 effort=2.0 velocity=3.1415
- joint joint2: limit lower=0.0 upper=2.9670597283903604 effort=60.0 velocity=3.1415 -> lower=0.0 upper=2.9670597283903604 effort=23.0 velocity=3.1415
- joint joint3: limit lower=-2.8797932657906435 upper=0.0 effort=30.0 velocity=3.1415 -> lower=-2.8797932657906435 upper=0.0 effort=10.0 velocity=3.1415
- joint joint4: limit lower=-1.5184364492350666 upper=1.5184364492350666 effort=30.0 velocity=3.1415 -> lower=-1.5184364492350666 upper=1.5184364492350666 effort=4.0 velocity=3.1415
- joint joint5: limit lower=-1.3439035240356338 upper=1.3439035240356338 effort=30.0 velocity=3.1415 -> lower=-1.3439035240356338 upper=1.3439035240356338 effort=4.0 velocity=3.1415
- joint joint6: limit lower=-2.792526803190927 upper=2.792526803190927 effort=30.0 velocity=3.1415 -> lower=-2.792526803190927 upper=2.792526803190927 effort=4.0 velocity=3.1415
